File: boomerang/boomerang.sch (EAGLE design)
At the start: 11 parts, among them IC1 WS2811-SOP8

Commit message: nicer :)
Parts:
- removed JP1: (no value), adafruit:PINHD-2X4
- removed PAD3, PAD4, PAD5, PAD6: (no value), wirepad:SMD2
- added BGND, BO, GGND, RGND: (no value), wirepad:SMD2
- added X3: 87438-06, con-molex:87438-06
- renumbered PAD1 to RO, PAD2 to GO
Connections:
- net N$1 renamed R
- net N$2 renamed G
- net N$3 renamed B
- net N$6 renamed GO
- net N$7 renamed RO
- removed net N$10: IC1.DO, JP1.8
- removed net N$5: IC1.DIN, JP1.7
- removed net N$9: PAD3.P, Q3.S
- new net BO: BO.P, Q3.S
- new net DIN: IC1.DIN, X3-3.S
- new net DO: IC1.DO, X3-4.S
- net 3V3: now also X3-1.S; no longer JP1.5, JP1.6
- net GND: now also BGND.P, GGND.P, RGND.P, X3-5.S, X3-6.S; no longer JP1.3, JP1.4, PAD4.P, PAD5.P, PAD6.P
- net VCC: now also X3-2.S; no longer JP1.1, JP1.2
Other:
- moved on the sheet: Q3
