File: boomerang/boomerangv2.brd (EAGLE design)
At the start: 136.9 x 62.2 mm, 11 parts, among them IC1 WS2811-SOP8, X3 87438-06

Commit message: foo
Parts:
- removed X3: 87438-06, con-molex:87438-06
- added X1, X2: 87438-05, con-molex:87438-05
- moved Q1 116.7 mm to (-5.08, -8.57), turned to 150 degrees
- moved Q3 108.3 mm to (-4.76, 8.57), turned to 30 degrees
- moved GGND 105.1 mm to (11.1, 2.00)
- moved GO 105.1 mm to (11.1, -2.00)
- moved RGND 104.4 mm to (-4.45, -11.4), turned to 150 degrees
- moved BGND 103.9 mm to (-7.94, 9.53), turned to 30 degrees
- moved BO 103.9 mm to (-3.81, 11.7), turned to 30 degrees
- moved RO 103.9 mm to (-7.94, -9.37), turned to 330 degrees
- moved IC1 103.7 mm to (1.91, 0.00)
- moved Q2 102.3 mm to (8.89, 0.00), turned to 270 degrees
Connections:
- net 3V3: now also X1.1, X2.1; no longer X3.1
- net DIN: now also X1.3; no longer X3.3
- net DO: now also X2.3; no longer X3.4
- net GND: now also X1.4, X1.5, X2.4, X2.5; no longer X3.5, X3.6
- net VCC: now also X1.2, X2.2; no longer X3.2
Routing:
- net GND: track 51.2 -> 0.00 mm
- net 3V3: track 22.2 -> 53.8 mm
- net RO: track 19.7 -> 3.41 mm
- net R: track 8.46 -> 20.1 mm
- net B: track 2.27 -> 8.96 mm
- net GO: track 7.35 -> 3.49 mm
- net BO: track 6.72 -> 3.83 mm
- net VCC: track 11.0 -> 13.1 mm
- net DIN: track 7.70 -> 9.79 mm
- net DO: track 5.56 -> 3.66 mm
- net G: track 8.34 -> 9.08 mm
Other:
- board size 136.9 x 62.2 mm -> 54.1 x 59.6 mm
- board text removed: "B+"
- board text removed: "B-"
- board text removed: "G+"
- board text removed: "G-"
- board text removed: "R+"
- board text removed: "R-"
