File: boomerangSATA/boomerang.sch (EAGLE design)
At the start: 12 parts

Commit message: updated SATA - connector part in library used
Connections:
- net GND: now also J1.GND3; no longer J1.VCC
- net VCC: now also J1.VCC2; no longer J1.GND
Changed lines of the file:
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@@
 </segment>
 <segment>
-<pinref part="J1" gate="G$1" pin="GND1"/>
-<wire x1="81.28" y1="0" x2="83.82" y2="0" width="0.1524" layer="91"/>
+<pinref part="J1" gate="G$1" pin="GND3"/>
 <label x="93.98" y="0" size="1.778" layer="95"/>
 <pinref part="J1" gate="G$1" pin="GND2"/>
-<wire x1="83.82" y1="0" x2="86.36" y2="0" width="0.1524" layer="91"/>
+<wire x1="81.28" y1="0" x2="86.36" y2="0" width="0.1524" layer="91"/>
 <wire x1="86.36" y1="0" x2="99.06" y2="0" width="0.1524" layer="91"/>
 <wire x1="81.28" y1="2.54" x2="86.36" y2="2.54" width="0.1524" layer="91"/>
 <wire x1="86.36" y1="2.54" x2="86.36" y2="0" width="0.1524" layer="91"/>
-<pinref part="J1" gate="G$1" pin="VCC"/>
-<wire x1="81.28" y1="10.16" x2="60.96" y2="10.16" width="0.1524" layer="91"/>
-<wire x1="60.96" y1="10.16" x2="60.96" y2="0" width="0.1524" layer="91"/>
-<wire x1="60.96" y1="0" x2="81.28" y2="0" width="0.1524" layer="91"/>
 </segment>
 <segment>
@@
 <wire x1="167.64" y1="22.86" x2="167.64" y2="15.24" width="0.1524" layer="91"/>
 <pinref part="C-RO" gate="G$1" pin="2"/>
+</segment>
+<segment>
+<pinref part="J1" gate="G$1" pin="GND1"/>
+<wire x1="81.28" y1="10.16" x2="99.06" y2="10.16" width="0.1524" layer="91"/>
+<label x="93.98" y="10.16" size="1.778" layer="95"/>
 </segment>
 </net>
@@
 <net name="VCC" class="0">
 <segment>
-<pinref part="J1" gate="G$1" pin="VCC1"/>
-<wire x1="81.28" y1="12.7" x2="99.06" y2="12.7" width="0.1524" layer="91"/>
-<label x="93.98" y="12.7" size="1.778" layer="95"/>
-<wire x1="81.28" y1="12.7" x2="55.88" y2="12.7" width="0.1524" layer="91"/>
-<wire x1="55.88" y1="12.7" x2="55.88" y2="-2.54" width="0.1524" layer="91"/>
-<pinref part="J1" gate="G$1" pin="GND"/>
-<wire x1="55.88" y1="-2.54" x2="81.28" y2="-2.54" width="0.1524" layer="91"/>
+<pinref part="J1" gate="G$1" pin="VCC2"/>
 <wire x1="81.28" y1="-2.54" x2="99.06" y2="-2.54" width="0.1524" layer="91"/>
+<label x="93.98" y="-2.54" size="1.778" layer="95"/>
 </segment>
 <segment>
@@
 <label x="165.1" y="38.1" size="1.778" layer="95" rot="R270"/>
 </segment>
+<segment>
+<pinref part="J1" gate="G$1" pin="VCC1"/>
+<wire x1="81.28" y1="12.7" x2="99.06" y2="12.7" width="0.1524" layer="91"/>
+<label x="93.98" y="12.7" size="1.778" layer="95"/>
+</segment>
 </net>
