File: hub/sata-hub3.brd (EAGLE design)
At the start: 100 x 80 mm, 3 parts

Commit message: .
Other:
- board size 100 x 80 mm -> 44.1 x 32.2 mm
Changed lines of the file:
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@@
 <board>
 <plain>
-<wire x1="0" y1="0" x2="100" y2="0" width="0" layer="20"/>
-<wire x1="100" y1="0" x2="100" y2="80" width="0" layer="20"/>
-<wire x1="100" y1="80" x2="0" y2="80" width="0" layer="20"/>
-<wire x1="0" y1="80" x2="0" y2="0" width="0" layer="20"/>
 <wire x1="22.5425" y1="45.87875" x2="42.2275" y2="57.30875" width="0" layer="20"/>
 <wire x1="42.2275" y1="57.30875" x2="47.78375" y2="57.30875" width="0" layer="20"/>
