File: diytextool/diytextool.brd (EAGLE design)
At the start: 12 parts

Commit message: foo
Parts:
- removed C-BO, C-GO, C-RO: (no value), pinhead:1X02M
- removed C1, C2: 100nF, resistor:C0603
- removed J1: (no value), dan-pc:SATA7-RA
- removed Q1, Q2, Q3: (no value), adafruit:SOT23
- removed U$2: LM3480IM4, SparkFun-PowerIC:SOT23-3
- added JP1: ISP, pinhead-2:2X03SMD
- moved U$1 32.5 mm to (33.0, 22.9), turned to 90 degrees
- moved R1 14.3 mm to (14.0, 15.2), turned to 180 degrees
Connections:
- removed net B: Q3.1, U$1.3
- removed net BO: C-BO.1, Q3.2
- removed net G: Q2.1, U$1.2
- removed net GO: C-GO.1, Q2.2
- removed net R: Q1.1, U$1.6
- removed net RES: R1.1, U$1.1
- removed net RO: C-RO.1, Q1.2
- removed net SCL: J1.5, U$1.7
- removed net SDA: J1.4, U$1.5
- removed net VCC: C2.1, J1.1, J1.7, Q1.3, Q2.3, Q3.3, U$2.2
- removed net VCC_GOOD: C1.1, R1.2, U$1.8, U$2.1
- new net +5V: JP1.2, R1.2, U$1.8
- new net N$2: JP1.5, R1.1, U$1.1
- new net N$6: JP1.4, U$1.5
- new net N$7: JP1.3, U$1.7
- new net N$8: JP1.1, U$1.6
- net GND: now also JP1.6; no longer C-BO.2, C-GO.2, C-RO.2, C1.2, C2.2, J1.2, J1.3, J1.6, U$2.3
Routing:
- net N$2: track 0.00 -> 46.0 mm
- net GND: track 0.00 -> 26.9 mm
- net VCC: track 25.3 -> 0.00 mm
- net +5V: track 0.00 -> 22.8 mm
- net N$8: track 0.00 -> 22.0 mm
- net N$6: track 0.00 -> 20.0 mm
- net N$7: track 0.00 -> 13.9 mm
- net VCC_GOOD: track 12.2 -> 0.00 mm
- net SCL: track 8.86 -> 0.00 mm
- net SDA: track 5.98 -> 0.00 mm
- net G: track 5.95 -> 0.00 mm
- net B: track 4.00 -> 0.00 mm
- net R: track 3.88 -> 0.00 mm
- net RES: track 3.51 -> 0.00 mm
Other:
- board outline added: 29.8 x 14.9 mm
