File: xmega/atxmega_e5.brd (EAGLE design)
At the start: 43.5 x 34.6 mm, 41 parts, among them IC2 ULN2003AD, M1_GND WIREPAD2,15/1,0, M1_VCC WIREPAD2,15/1,0, M2_GND WIREPAD2,15/1,0, M2_VCC WIREPAD2,15/1,0, M3_GND WIREPAD2,15/1,0, M3_VCC WIREPAD2,15/1,0, M4_GND WIREPAD2,15/1,0, M4_VCC WIREPAD2,15/1,0, M5_GND WIREPAD2,15/1,0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

Commit message: new revision (ready for OSHpark)
Parts:
- added LED4: (no value), LEDs:0805LED
- added O1, O2: 18pF, resistor:C0603K
- added R7: 470, resistor:R0603
- added U$1: CRYSTALABM7, atmega32u4-breakout-v3:ABM7
- moved C5 0.32 mm to (42.0, 16.9)
- moved IC2 0.24 mm to (37.1, 22.2)
- moved R4 0.24 mm to (19.1, 16.7)
- moved C7 0.16 mm to (19.1, 20.2)
Connections:
- new net N$1: O1.1, U$1.P$2, U1.20
- new net N$17: LED4.A, R7.1
- new net N$8: O2.1, U$1.P$1, U1.19
- net GND: now also LED4.C, O1.2, O2.2
- net N$11: now also R7.2
Routing:
- net N$8: track 0.00 -> 14.3 mm, vias 0 -> 1
- net N$1: track 0.00 -> 11.5 mm, vias 0 -> 1
- net N$21: track 20.2 -> 23.8 mm
- net N$11: track 14.5 -> 16.5 mm
- net N$17: track 0.00 -> 1.81 mm
- net GND: track 11.0 -> 9.87 mm, vias 37 -> 36
