File: xmega/atxmega_e5.sch (EAGLE design)
At the start: 41 parts, among them IC2 ULN2003AD, M1_GND WIREPAD2,15/1,0, M1_VCC WIREPAD2,15/1,0, M2_GND WIREPAD2,15/1,0, M2_VCC WIREPAD2,15/1,0, M3_GND WIREPAD2,15/1,0, M3_VCC WIREPAD2,15/1,0, M4_GND WIREPAD2,15/1,0, M4_VCC WIREPAD2,15/1,0, M5_GND WIREPAD2,15/1,0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

Commit message: new revision (ready for OSHpark)
Parts:
- added LED4: (no value), LEDs:LED0805LED
- added O1, O2: 18pF, resistor:C-EUC0603K
- added R7: 470, resistor:R-EU_R0603
- added U$1: CRYSTALABM7, atmega32u4-breakout-v3:CRYSTALABM7
Connections:
- new net N$1: O1.1, U$1.2, U1.PR0/XTAL2/TOSC2/CLKOUT/EVOUT/RTCOUT/AC1OUT
- new net N$17: LED4.A, R7.1
- new net N$8: O2.1, U$1.1, U1.PR1/XTAL1/TOSC1/EXTCLK/AC0OUT
- net GND: now also LED4.C, O1.2, O2.2
- net N$11: now also R7.2
Other:
- moved on the sheet: SJ1, SJ2, X1
Changed lines of the file:
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@@
 <part name="LED3" library="LEDs" deviceset="LED" device="0805LED"/>
 <part name="GND16" library="supply1" deviceset="GND" device=""/>
+<part name="U$1" library="atmega32u4-breakout-v3" deviceset="CRYSTAL" device="ABM7"/>
+<part name="O1" library="resistor" deviceset="C-EU" device="C0603K" value="18pF"/>
+<part name="O2" library="resistor" deviceset="C-EU" device="C0603K" value="18pF"/>
+<part name="GND15" library="supply1" deviceset="GND" device=""/>
+<part name="R7" library="resistor" deviceset="R-EU_" device="R0603" value="470"/>
+<part name="LED4" library="LEDs" deviceset="LED" device="0805LED"/>
+<part name="GND17" library="supply1" deviceset="GND" device=""/>
 </parts>
 <sheets>
@@
 </instance>
 <instance part="73831" gate="G$1" x="60.96" y="50.8"/>
-<instance part="X1" gate="G$1" x="10.16" y="15.24" smashed="yes" rot="R180">
-<attribute name="NAME" x="12.7" y="3.81" size="1.778" layer="95" font="vector" rot="R180"/>
-</instance>
-<instance part="SJ1" gate="1" x="48.26" y="15.24" smashed="yes">
-<attribute name="NAME" x="45.72" y="17.78" size="1.778" layer="95"/>
-</instance>
-<instance part="SJ2" gate="1" x="40.64" y="17.78" smashed="yes">
-<attribute name="NAME" x="38.1" y="20.32" size="1.778" layer="95"/>
+<instance part="X1" gate="G$1" x="43.18" y="2.54" smashed="yes" rot="R180">
+<attribute name="NAME" x="45.72" y="-8.89" size="1.778" layer="95" font="vector" rot="R180"/>
+</instance>
+<instance part="SJ1" gate="1" x="81.28" y="2.54" smashed="yes">
+<attribute name="NAME" x="78.74" y="5.08" size="1.778" layer="95"/>
+</instance>
+<instance part="SJ2" gate="1" x="73.66" y="5.08" smashed="yes">
+<attribute name="NAME" x="71.12" y="7.62" size="1.778" layer="95"/>
 </instance>
 <instance part="U$2" gate="G$1" x="162.56" y="45.72" rot="R180"/>
@@
 <instance part="LED3" gate="G$1" x="147.32" y="132.08" rot="R270"/>
 <instance part="GND16" gate="1" x="139.7" y="124.46"/>
+<instance part="U$1" gate="G$1" x="160.02" y="88.9" smashed="yes" rot="R90">
+<attribute name="VALUE" x="160.02" y="91.44" size="1.778" layer="96"/>
+</instance>
+<instance part="O1" gate="G$1" x="152.4" y="91.44" smashed="yes" rot="R270">
+<attribute name="NAME" x="153.924" y="91.821" size="1.778" layer="95"/>
+<attribute name="VALUE" x="143.764" y="91.821" size="1.778" layer="96"/>
+</instance>
+<instance part="O2" gate="G$1" x="152.4" y="86.36" smashed="yes" rot="R270">
+<attribute name="NAME" x="153.924" y="84.201" size="1.778" layer="95"/>
+<attribute name="VALUE" x="143.764" y="84.201" size="1.778" layer="96"/>
+</instance>
+<instance part="GND15" gate="1" x="139.7" y="81.28"/>
+<instance part="R7" gate="G$1" x="40.64" y="35.56" rot="MR180"/>
+<instance part="LED4" gate="G$1" x="30.48" y="30.48"/>
+<instance part="GND17" gate="1" x="30.48" y="22.86"/>
 </instances>
 <busses>
@@
 <segment>
 <pinref part="X1" gate="G$1" pin="5"/>
-<wire x1="15.24" y1="20.32" x2="33.02" y2="20.32" width="0.1524" layer="91"/>
-<label x="20.32" y="20.32" size="1.778" layer="95"/>
+<wire x1="48.26" y1="7.62" x2="66.04" y2="7.62" width="0.1524" layer="91"/>
+<label x="53.34" y="7.62" size="1.778" layer="95"/>
 </segment>
 <segment>
@@
 <pinref part="GND16" gate="1" pin="GND"/>
 </segment>
+<segment>
+<pinref part="O1" gate="G$1" pin="2"/>
+<wire x1="147.32" y1="91.44" x2="139.7" y2="91.44" width="0.1524" layer="91"/>
+<wire x1="139.7" y1="91.44" x2="139.7" y2="86.36" width="0.1524" layer="91"/>
+<pinref part="O2" gate="G$1" pin="2"/>
+<wire x1="139.7" y1="86.36" x2="139.7" y2="83.82" width="0.1524" layer="91"/>
+<wire x1="147.32" y1="86.36" x2="139.7" y2="86.36" width="0.1524" layer="91"/>
+<pinref part="GND15" gate="1" pin="GND"/>
+</segment>
+<segment>
+<pinref part="LED4" gate="G$1" pin="C"/>
+<pinref part="GND17" gate="1" pin="GND"/>
+<wire x1="30.48" y1="25.4" x2="30.48" y2="27.94" width="0.1524" layer="91"/>
+</segment>
 </net>
 <net name="VIN" class="0">
 <segment>
 <pinref part="X1" gate="G$1" pin="1"/>
-<wire x1="15.24" y1="10.16" x2="33.02" y2="10.16" width="0.1524" layer="91"/>
-<label x="20.32" y="10.16" size="1.778" layer="95"/>
+<wire x1="48.26" y1="-2.54" x2="66.04" y2="-2.54" width="0.1524" layer="91"/>
+<label x="53.34" y="-2.54" size="1.778" layer="95"/>
 </segment>
 <segment>
@@
 <segment>
 <pinref part="X1" gate="G$1" pin="4"/>
-<wire x1="15.24" y1="17.78" x2="35.56" y2="17.78" width="0.1524" layer="91"/>
-<label x="20.32" y="17.78" size="1.778" layer="95"/>
+<wire x1="48.26" y1="5.08" x2="68.58" y2="5.08" width="0.1524" layer="91"/>
+<label x="53.34" y="5.08" size="1.778" layer="95"/>
 <pinref part="SJ2" gate="1" pin="1"/>
 </segment>
@@
 <segment>
 <pinref part="X1" gate="G$1" pin="3"/>
-<wire x1="15.24" y1="15.24" x2="43.18" y2="15.24" width="0.1524" layer="91"/>
-<label x="20.32" y="15.24" size="1.778" layer="95"/>
+<wire x1="48.26" y1="2.54" x2="76.2" y2="2.54" width="0.1524" layer="91"/>
+<label x="53.34" y="2.54" size="1.778" layer="95"/>
 <pinref part="SJ1" gate="1" pin="1"/>
 </segment>
@@
 <segment>
 <pinref part="X1" gate="G$1" pin="2"/>
-<wire x1="15.24" y1="12.7" x2="33.02" y2="12.7" width="0.1524" layer="91"/>
-<label x="20.32" y="12.7" size="1.778" layer="95"/>
+<wire x1="48.26" y1="0" x2="66.04" y2="0" width="0.1524" layer="91"/>
+<label x="53.34" y="0" size="1.778" layer="95"/>
 </segment>
 </net>
@@
 <segment>
 <pinref part="SJ2" gate="1" pin="2"/>
-<wire x1="45.72" y1="17.78" x2="66.04" y2="17.78" width="0.1524" layer="91"/>
-<label x="55.88" y="17.78" size="1.778" layer="95"/>
+<wire x1="78.74" y1="5.08" x2="99.06" y2="5.08" width="0.1524" layer="91"/>
+<label x="88.9" y="5.08" size="1.778" layer="95"/>
 </segment>
 <segment>
@@
 <segment>
 <pinref part="SJ1" gate="1" pin="2"/>
-<wire x1="53.34" y1="15.24" x2="66.04" y2="15.24" width="0.1524" layer="91"/>
-<label x="55.88" y="15.24" size="1.778" layer="95"/>
+<wire x1="86.36" y1="2.54" x2="99.06" y2="2.54" width="0.1524" layer="91"/>
+<label x="88.9" y="2.54" size="1.778" layer="95"/>
 </segment>
 <segment>
@@
 <wire x1="48.26" y1="45.72" x2="48.26" y2="43.18" width="0.1524" layer="91"/>
 <wire x1="48.26" y1="43.18" x2="43.18" y2="43.18" width="0.1524" layer="91"/>
+<pinref part="R7" gate="G$1" pin="2"/>
+<wire x1="48.26" y1="43.18" x2="48.26" y2="35.56" width="0.1524" layer="91"/>
+<wire x1="48.26" y1="35.56" x2="45.72" y2="35.56" width="0.1524" layer="91"/>
+<junction x="48.26" y="43.18"/>
 </segment>
 </net>
@@
 </segment>
 </net>
+<net name="N$1" class="0">
+<segment>
+<pinref part="O1" gate="G$1" pin="1"/>
+<pinref part="U$1" gate="G$1" pin="2"/>
+<wire x1="154.94" y1="91.44" x2="160.02" y2="91.44" width="0.1524" layer="91"/>
+<wire x1="160.02" y1="91.44" x2="170.18" y2="91.44" width="0.1524" layer="91"/>
+<wire x1="170.18" y1="91.44" x2="170.18" y2="96.52" width="0.1524" layer="91"/>
+<pinref part="U1" gate="G$1" pin="PR0/XTAL2/TOSC2/CLKOUT/EVOUT/RTCOUT/AC1OUT"/>
+<wire x1="170.18" y1="96.52" x2="177.8" y2="96.52" width="0.1524" layer="91"/>
+</segment>
+</net>
+<net name="N$8" class="0">
+<segment>
+<pinref part="U1" gate="G$1" pin="PR1/XTAL1/TOSC1/EXTCLK/AC0OUT"/>
+<wire x1="177.8" y1="93.98" x2="172.72" y2="93.98" width="0.1524" layer="91"/>
+<wire x1="172.72" y1="93.98" x2="172.72" y2="86.36" width="0.1524" layer="91"/>
+<pinref part="U$1" gate="G$1" pin="1"/>
+<wire x1="172.72" y1="86.36" x2="160.02" y2="86.36" width="0.1524" layer="91"/>
+<pinref part="O2" gate="G$1" pin="1"/>
+<wire x1="160.02" y1="86.36" x2="154.94" y2="86.36" width="0.1524" layer="91"/>
+</segment>
+</net>
+<net name="N$17" class="0">
+<segment>
+<pinref part="R7" gate="G$1" pin="1"/>
+<pinref part="LED4" gate="G$1" pin="A"/>
+<wire x1="30.48" y1="35.56" x2="35.56" y2="35.56" width="0.1524" layer="91"/>
+</segment>
+</net>
